File: hw/WHL0137-LS/LED_ring.kicad_sch (KiCad schematic)
At the start: 43 parts, among them U1 IS31FL3236A

Commit message: Some layout
Parts:
- removed R1: 100k, Resistor_SMD:R_0805_2012Metric, symbol Device:R
- renumbered D5 to D10, D14 to D11, D4 to D12, D15 to D13, D3 to D14, D16 to D15, D2 to D16, D1 to D18, D18 to D19, D9 to D2, D19 to D20, D28 to D21, D20 to D22, D29 to D23, D21 to D24, D30 to D25, D22 to D26, D31 to D27, D23 to D28, D32 to D29, D10 to D3, D24 to D30, D33 to D31, D25 to D32, D34 to D33, D26 to D34, D27 to D36, D36 to D37, D8 to D4, D11 to D5, D7 to D6, D12 to D7, D6 to D8, D13 to D9, R2 to R3
Other:
- moved on the sheet: D10, D11, D12, D13, D14, D15, D16, D17, D18, D19, D2, D3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
