File: hw/WHL0137-LS/WHL0137-LS.kicad_pcb (KiCad board)
At the start: 4 copper layers, 103.9 x 117.2 mm, 89 parts, among them J1 Conn_01x05, U1 IS31FL3236A, U2 IS31FL3236A

Commit message: misc changes
Parts:
- removed TP1, TP2: TestPoint, TestPoint:TestPoint_Pad_D2.5mm
- moved C2 2.60 mm to (-23.0, -61.8), turned to 90 degrees
- moved C4 2.10 mm to (23.0, -61.8), turned to 90 degrees
- moved R1 1.74 mm to (18.2, -63.8), turned to 0 degrees
- moved R3 1.10 mm to (-18.0, -63.2)
- moved C3 0.89 mm to (21.0, -61.8), turned to 90 degrees
- moved C1 0.34 mm to (-21.0, -61.8), turned to 90 degrees
Routing:
- net GND: track 14.1 -> 43.7 mm, vias 7 -> 5
- net +5V: track 18.5 -> 14.4 mm
- net /led_driver_1/R_EXT: track 8.65 -> 7.69 mm
- net /led_driver_2/R_EXT: track 7.74 -> 6.81 mm
- net Net-(D55-Pad1): track 137.2 -> 136.4 mm
- net Net-(D25-Pad1): track 87.8 -> 87.1 mm
Other:
- board size 103.9 x 117.2 mm -> 106 x 118.2 mm
- board text added: "SCL"
- board text added: "SDA"
- board text added: "SDB"
