File: hw/WHL0137-LS/led_driver_1.kicad_sch (KiCad schematic)
At the start: 42 parts, among them U1 IS31FL3236A

Commit message: misc changes
Other:
- note added: "JP1/JP2 Configurations --------------- JP1 1-2: AD set to 10 JP1 2-3: AD set to 01 JP2 1-2: AD set to 11 JP2 2-3: AD set to 00"
Changed lines of the file:
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@@
     (stroke (width 0) (type default) (color 0 0 0 0))
   )
-  (wire (pts (xy 111.76 66.04) (xy 120.65 66.04))
+  (wire (pts (xy 114.3 66.04) (xy 120.65 66.04))
     (stroke (width 0) (type default) (color 0 0 0 0))
   )
@@
     (stroke (width 0) (type default) (color 0 0 0 0))
   )
-  (wire (pts (xy 111.76 71.12) (xy 120.65 71.12))
+  (wire (pts (xy 114.3 71.12) (xy 120.65 71.12))
     (stroke (width 0) (type default) (color 0 0 0 0))
   )
@@
     (stroke (width 0) (type default) (color 0 0 0 0))
   )
-  (wire (pts (xy 111.76 68.58) (xy 120.65 68.58))
+  (wire (pts (xy 114.3 68.58) (xy 120.65 68.58))
     (stroke (width 0) (type default) (color 0 0 0 0))
   )
@@
     (stroke (width 0) (type default) (color 0 0 0 0))
   )
-  (image (at 245.11 40.64)
+  (image (at 262.89 25.4)
     (data
       iVBORw0KGgoAAAANSUhEUgAAAaQAAADdCAIAAAB7dJHfAAAAA3NCSVQICAjb4U/gAAAACXBIWXMA
@@
     )
   )
+  (text "JP1/JP2 Configurations\n---------------\nJP1 1-2: AD set to 10\nJP1 2-3: AD set to 01\nJP2 1-2: AD set to 11\nJP2 2-3: AD set to 00"
+    (at 224.79 60.96 0)
+    (effects (font (size 1.27 1.27)) (justify left bottom))
+  )
   (label "R_EXT" (at 161.29 76.2 0)
     (effects (font (size 1.27 1.27)) (justify left bottom))
@@
     (effects (font (size 1.27 1.27)) (justify left bottom))
   )
-  (hierarchical_label "SCL" (shape input) (at 111.76 68.58 180)
+  (hierarchical_label "SCL" (shape input) (at 114.3 68.58 180)
     (effects (font (size 1.27 1.27)) (justify right))
   )
-  (hierarchical_label "SDB" (shape input) (at 111.76 71.12 180)
+  (hierarchical_label "SDB" (shape input) (at 114.3 71.12 180)
     (effects (font (size 1.27 1.27)) (justify right))
   )
-  (hierarchical_label "SDA" (shape bidirectional) (at 111.76 66.04 180)
+  (hierarchical_label "SDA" (shape bidirectional) (at 114.3 66.04 180)
     (effects (font (size 1.27 1.27)) (justify right))
   )
