File: hw/WHL0137-LS/led_driver_2.kicad_sch (KiCad schematic)
At the start: 42 parts, among them U2 IS31FL3236A

Commit message: misc changes
Other:
- note added: "JP3/JP4 Configurations --------------- JP3 1-2: AD set to 10 JP3 2-3: AD set to 01 JP4 1-2: AD set to 11 JP4 2-3: AD set to 00"
Changed lines of the file:
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@@
     (stroke (width 0) (type default) (color 0 0 0 0))
   )
-  (image (at 243.84 36.83)
+  (image (at 261.62 26.67)
     (data
       iVBORw0KGgoAAAANSUhEUgAAAaQAAADdCAIAAAB7dJHfAAAAA3NCSVQICAjb4U/gAAAACXBIWXMA
@@
     )
   )
+  (text "JP3/JP4 Configurations\n---------------\nJP3 1-2: AD set to 10\nJP3 2-3: AD set to 01\nJP4 1-2: AD set to 11\nJP4 2-3: AD set to 00"
+    (at 224.79 57.15 0)
+    (effects (font (size 1.27 1.27)) (justify left bottom))
+  )
   (label "SDA" (at 190.5 46.99 90)
